File: corne-pcb_left/corne-pcb_left.kicad_pcb (KiCad board)
At the start: 2 copper layers, 46 parts, among them SW1 SW_SPST, U1 Nice_Nano_V2, U2 TRRS

Commit message: add encoder to left
Parts:
- added D22: Diode, ScottoKeebs_Components:Diode_SOD-123, B.Cu at (172.5, 99.0)
- added SW2: RotaryEncoder_Switch, ScottoKeebs_Scotto:Encoder_EC11_MX, F.Cu at (165.0, 92.0)
- moved SW1 31.6 mm to (199.0, 90.8)
- moved U2 30.8 mm to (201.1, 81.5)
- renumbered D5 to D1, D7 to D10, D9 to D11, D10 to D12, D17 to D13, D18 to D14, D14 to D15, D13 to D16, D15 to D17, D16 to D18, D6 to D2, D2 to D3, D1 to D4, D3 to D5, D4 to D6, D11 to D7, D12 to D8, D8 to D9, S5 to S1, S7 to S10, S9 to S11, S10 to S12, S17 to S13, S18 to S14, S14 to S15, S13 to S16, S15 to S17, S16 to S18, S6 to S2, S2 to S3, S1 to S4, S3 to S5, S4 to S6, S11 to S7, S12 to S8, S8 to S9
Connections:
- S19 pad 1: Column 3 -> unconnected-(S19-Pad1)
- S20 pad 1: Column 4 -> unconnected-(S20-Pad1)
- S21 pad 1: Column 5 -> unconnected-(S21-Pad1)
- U1 pad 19: unconnected-(U1-20-Pad19) -> EncoderB
- U1 pad 20: unconnected-(U1-21-Pad20) -> EncoderA
