File: corne-pcb_left/corne-pcb_left.kicad_sch (KiCad schematic)
At the start: 47 parts, among them SW1 SW_SPST, SW2 RotaryEncoder_Switch, U1 Nice_Nano_V2, U2 TRRS

Commit message: add encoder to left
Parts:
- added D22: Diode, ScottoKeebs_Components:Diode_SOD-123, symbol ScottoKeebs:Placeholder_Diode
Connections:
- net Column 3: no longer S19.1
- net Column 4: no longer S20.1
- net Column 5: no longer S21.1
- net GND: now also SW2.C
- net Row 2: now also SW2.S2
- net Row 3: now also D22.1 (K)
- net EncoderA: now reaches SW2.A
- net EncoderA: now also U1.20 (21)
- net EncoderB: now reaches SW2.B
- net EncoderB: now also U1.19 (20)
- net at SW2.S1: now also D22.2 (A)
Other:
- moved on the sheet: SW2, U2
